File: PCB/docDongle/schematics/MB1293C/Schematic.kicad_sch (KiCad schematic)
At the start: 65 parts

Commit message: a
Parts:
- removed D1, D2, D3: (no value), symbol Schematic-altium-import:3_LED
- removed R3: (no value), symbol Schematic-altium-import:1_RES
- removed R4, R5, R6: (no value), symbol Schematic-altium-import:3_RES
- removed SC1, SC2, SC3, SC4: (no value), symbol Schematic-altium-import:0_Shield Clip_A 3.9x1.1x1.28
- removed SH1: (no value), symbol Schematic-altium-import:0_Shield
- removed SW1: (no value), symbol Schematic-altium-import:1_SW-PB_1
Other:
- note removed: "Socket for Metallic Shield"
