File: PCB/watch/watch.kicad_sch (KiCad schematic)
At the start: 0 parts

Commit message: a
Parts:
- added C1, C12, C19, C2, C20, C4, C8: (no value), symbol Schematic-altium-import:1_CAP_NPOL
- added C10, C17, C18, C22, C28, C29, C6, C9: (no value), symbol Schematic-altium-import:0_CAP_NPOL
- added C15, C16: (no value), symbol Schematic-altium-import:3_CAP_NPOL
- added C21, C23, C24, C25, C26, C27, C3, C30, C7: (no value), symbol Schematic-altium-import:2_CAP_NPOL
- added CN1: (no value), symbol Schematic-altium-import:0_HEADER_1X10
- added CN2: (no value), symbol Schematic-altium-import:0_mirrored_HEADER_1X10
- added CN3: (no value), symbol Schematic-altium-import:0_USB_1
- added CN4: (no value), symbol Schematic-altium-import:0_mirrored_HEADER_1X4
- added CN5: (no value), symbol Schematic-altium-import:0_mirrored_UFL
- added D4: (no value), symbol Schematic-altium-import:0_BAT54K
- added FLT1: (no value), symbol Schematic-altium-import:0_LFB182G45CGFD436
- added L1, L4, L6: (no value), symbol Schematic-altium-import:1_INDUCTOR_SMD_STDL
- added L2: (no value), symbol Schematic-altium-import:2_IND_74479777310A
- added L3: (no value), symbol Schematic-altium-import:1_IND_FCM1608KF-601T03
- added R1: (no value), symbol Schematic-altium-import:2_RES
- added R2: (no value), symbol Schematic-altium-import:0_RES
- added SB1, SB2, SB3, SB6: (no value), symbol Schematic-altium-import:0_Strap2
- added SB4: (no value), symbol Schematic-altium-import:1_Strap2
- added SB5: (no value), symbol Schematic-altium-import:3_Strap2
- added SW2: (no value), symbol Schematic-altium-import:3_mirrored_MLL1200S_TE
- added U1: (no value), symbol Schematic-altium-import:0_STM32WBxx_QFN48
- added U2: (no value), symbol Schematic-altium-import:0_mirrored_USBLC6-2
- added U3: (no value), symbol Schematic-altium-import:0_LD3985M33R
- added X1: (no value), symbol Schematic-altium-import:3_NX2016_32M
- added X2: (no value), symbol Schematic-altium-import:0_NX2012_32K768
Connections:
- new net: C29.1, CN5.1 (X), L4.2
- new net: C22.1, L3.2, U1.8 (VDDA/VREF+)
- new net: C4.1, C8.1, FLT1.3 (I/O)
- new net: C4.2, C6.1, L1.1
- new net: C26.2, C27.2, SB4.2, U3.5 (VOUT)
- new net: C10.1, L2.1, SB1.1, U1.31 (VFBSMPS)
- new net: L2.2, U1.33 (VLXSMPS)
- new net: C28.1, C8.2, L4.1
- new net: C19.1, SB5.1, U1.20 (VDD/VDDT)
- new net: CN4.1, U1.26 (AT0)
- new net: CN4.2, U1.27 (AT1)
- new net: CN2.7, SB2.1, SB6.1
- new net: C25.2, U3.4 (BYPASS)
- new net: C17.1, U1.2 (PC14-OSC32_IN), X2.1 (OSC1)
- new net: U1.24 (OSC_OUT), X1.3 (OSC2)
- new net: U1.25 (OSC_IN), X1.1 (OSC1)
- new net: C18.1, U1.3 (PC15-OSC32_OUT), X2.2 (OSC2)
- new net: C12.1, D4.A, R1.2, U1.7 (NRST)
- new net: C3.2, FLT1.1 (I/O), L6.2
- new net: C30.2, L6.1, U1.21 (RF1)
- new net: CN3.3 (D+), U2.4
- new net: CN3.2 (D_-), U2.6
- new net 3V3: C1.2, C15.1, C16.1, C2.2, C20.2, C21.2, C9.1, CN1.6, L3.1, R1.1, SB1.2, SB3.1, SB4.1, SB5.2, SW2.2, U1.1 (VBAT), U1.23 (VDDRF), U1.34 (VDDSMPS), U1.35 (VDD), U1.40 (VDDUSB), U1.48 (VDD)
- new net 5V_USB: C23.2, C24.2, CN3.1 (VBUS), U2.5, U3.1 (VIN), U3.3 (CE)
- new net ANT: C7.2, L1.2
- new net BOOT0: R2.1, SB3.2, SW2.3, U1.4 (PH3-BOOT0)
- new net GND: C1.1, C10.2, C12.2, C15.2, C16.2, C17.2, C18.2, C19.2, C2.1, C20.1, C21.1, C22.2, C23.1, C24.1, C25.1, C26.1, C27.1, C28.2, C29.2, C3.1, C30.1, C6.2, C7.1, C9.2, CN1.1, CN2.9, CN3.0 (Shield), CN3.4 (GND), CN5.2 (Y), FLT1.2 (GND), R2.2, U1.22 (RF0), U1.32 (VSSSMPS), U1.49 (VSS_(ExPAD)), U2.2, U3.2 (VSS), X1.2, X1.4
- new net NRST: CN1.2, D4.K
- new net PA0: CN2.3, U1.9 (PA0)
- new net PA1: CN2.10, U1.10 (PA1)
- new net PA10: U1.36 (PA10)
- new net PA13: CN1.3, U1.39 (PA13-SWDIO)
- new net PA14: CN1.4, U1.41 (PA14-SWCLK)
- new net PA2: CN2.4, U1.11 (PA2)
- new net PA3: CN2.5, U1.12 (PA3)
- new net PA4: U1.13 (PA4)
- new net PA5: CN1.8, U1.14 (PA5)
- new net PA6: CN1.9, U1.15 (PA6)
- new net PA7: CN1.10, U1.16 (PA7)
- new net PA8: CN2.8, U1.17 (PA8)
- new net PA9: SB2.2, U1.18 (PA9)
- new net PB0: CN4.3, U1.28 (PB0)
- new net PB1: CN4.4, U1.29 (PB1)
- new net PB2: CN1.7, U1.19 (PB2)
- new net PB3: CN1.5, U1.43 (PB3-SWO)
- new net PB6: CN2.6, U1.46 (PB6)
- new net PB7: SB6.2, U1.47 (PB7)
- new net PB8: CN2.1, U1.5 (PB8)
- new net PB9: CN2.2, U1.6 (PB9)
- new net USB_N: U1.37 (PA11), U2.1
- new net USB_P: U1.38 (PA12), U2.3
- no-connect marks 0 -> 5
Other:
- note added: "${##}"
- note added: "${#}"
- note added: "${BOARD_ASSEMBLY_REVISION}"
- note added: "${BOARD_DOCUMENT_DATE}"
- note added: "${BOARD_NAME}"
- note added: "${BOARD_PCB_REVISION}"
- note added: "${BOARD_REFERENCE}"
- note added: "${TITLE}"
- note added: "${VARIANTNAME}"
- note added: "(Compents values will be updated after evaluation)"
- note added: "(default position)"
- note added: "(see AN3359 on www.st.com)"
- note added: "-"
- note added: "2.4GHz"
- note added: "50 Ohms Matching Network"
- note added: "A4"
- note added: "ADC"
- note added: "AT0"
- note added: "AT1"
- note added: "AT2"
- note added: "AT3"
- note added: "Antenna Matching Network"
- note added: "Antenna Matching Network (connected to UFL)"
- note added: "BOOT0 = "0""
- note added: "BOOT0 = "1""
- note added: "Band Pass Filter"
- note added: "Date:"
- note added: "Debug : Vref for STLink"
- note added: "Dongle USB : Vout (3V3)"
- note added: "GND"
- note added: "GPIO"
- note added: "I2C1_SCL"
- note added: "I2C1_SDA"
- note added: "LPUART1_RX"
- note added: "LPUART1_TX"
- note added: "Meander Antenna"
- note added: "Module : Vin (1V8 to 3V6)"
- note added: "NRST"
- note added: "PCB Antenna"
- note added: "Project:"
- note added: "Reference:"
- note added: "Revision:"
- note added: "SPI1_MISO"
- note added: "SPI1_MOSI"
- note added: "SPI1_NSS"
- note added: "SPI1_SCK"
- note added: "SWCLK"
- note added: "SWDIO"
- note added: "SWO"
- note added: "Sheet:"
- note added: "Size:"
- note added: "Title:"
- note added: "Variant:"
- note added: "WKUP"
- note added: "of"
- company: AJJCT -> (none)
- title: HealthWatch -> STM32WB55CG USB Dongle Schematic
